File: PCB/PCB-MTD.kicad_sch (KiCad schematic)
At the start: 22 parts, among them J1 Barrel_Jack_Switch, J9 Micro_SD_Card, U1 ESP32-S3-UNO, U2 R-78E5.0-1.0

Commit message: Add files via upload
Parts:
- added C3, C4, C5: 10uF, C_1206_3216Metric_Pad1.33x1.80mm_HandSolder, symbol Device:C
Connections:
- net +3.3V: now also C5.2
- net +5V: now also C3.1
- net 12VF: now also C4.1
- net GND: now also C3.2, C4.2, C5.1
- net +12V: no longer names the net of F1.2, J1.1
Other:
- moved on the sheet: F1, J1, U2
