File: PCB/PCB-MTD.kicad_sch (KiCad schematic)
At the start: 26 parts, among them J1 Barrel_Jack_Switch, J2 Screw_Terminal_01x02, J9 Micro_SD_Card, U1 ESP32-S3-UNO, U2 R-78E5.0-1.0

Commit message: Add files via upload
Parts:
- C1, C2: footprint C_1206_3216Metric_Pad1.33x1.80mm_HandSolder -> Capacitor_SMD:CP_Elec_6.3x5.4
Connections:
- net +3.3V: now also R2.1, R3.1, jumperD1.1 (Pin_1), jumperD1.3 (Pin_3), jumperD1.5 (Pin_5), jumperD2.1 (Pin_1), jumperD2.3 (Pin_3), jumperD2.5 (Pin_5)
- net +5V: no longer jumperD1.1 (Pin_1), jumperD1.3 (Pin_3), jumperD1.5 (Pin_5), jumperD2.1 (Pin_1), jumperD2.3 (Pin_3), jumperD2.5 (Pin_5)
- net SCL: now also LCD1.3 (Pin_3)
- net SDA: now also LCD1.4 (Pin_4)
Other:
- moved on the sheet: R2, R3

Commit message: fix wiring problems
Connections:
- net +5V: no longer U1.8 (v_in)
- net 12VF: now also U1.8 (v_in)
