File: PCB/_autosave-PCB-MTD.kicad_pcb (KiCad board)
At the start: 2 copper layers, 78.2 x 57.6 mm, 25 parts, among them J1 Barrel_Jack_Switch, J9 Micro_SD_Card, U1 ESP32-S3-UNO, U2 R-78E5.0-1.0

Commit message: Add files via upload
Routing:
- net GND: track 0.13 -> 53.9 mm
Other:
- board text removed: "${REFERENCE}"
Changed lines of the file:
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@@
 		(tags "Through hole pin header THT 1x03 2.54mm single row")
 		(property "Reference" "Servo-moteur1"
-			(at 2.95 1.69 0)
+			(at -0.17 12.56 0)
 			(layer "F.SilkS")
 			(effects
@@
 			(at 0 7.46 90)
 			(layer "F.Fab")
+			(hide yes)
 			(effects
 				(font
@@
 			(layer "F.Fab")
 		)
-		(fp_text user "${REFERENCE}"
-			(at 0 2.54 0)
-			(layer "F.Fab")
-			(effects
-				(font
-					(size 1 1)
-					(thickness 0.15)
-				)
-			)
-		)
 		(pad "1" thru_hole rect
 			(at 0 0 90)
@@
 			(at 0 22.86 0)
 			(layer "B.Fab")
+			(hide yes)
 			(effects
 				(font
@@
 		)
 		(property "Value" "4.7k"
-			(at 0 1.65 270)
+			(at 1.67 2.03 270)
 			(layer "F.Fab")
 			(effects
@@
 		(tags "resistor handsolder")
 		(property "Reference" "R1"
-			(at 0 -1.65 270)
+			(at -0.74 -1.65 270)
 			(layer "F.SilkS")
 			(effects
@@
 		)
 		(property "Value" "10k"
-			(at 0 1.65 270)
+			(at 1.56 1.58 270)
 			(layer "F.Fab")
 			(effects
@@
 		(tags "resistor handsolder")
 		(property "Reference" "R2"
-			(at 0 -1.65 180)
+			(at -2.09 -1.53 180)
 			(layer "F.SilkS")
 			(effects
@@
 		(tags "capacitor handsolder")
 		(property "Reference" "C5"
-			(at 0 -1.85 0)
+			(at -4.39 2.48 0)
 			(layer "F.SilkS")
+			(hide yes)
 			(effects
 				(font
@@
 		(tags "Through hole pin header THT 1x04 2.54mm single row")
 		(property "Reference" "LCD1"
-			(at 0 -2.38 90)
+			(at 0.33 -2.86 90)
 			(layer "F.SilkS")
 			(effects
@@
 			(at 0 10 90)
 			(layer "F.Fab")
+			(hide yes)
 			(effects
 				(font
@@
 		(layer "Edge.Cuts")
 	)
-	(gr_text "${REFERENCE}"
-		(at 106.98 75.29 180)
-		(layer "B.Fab")
-		(effects
-			(font
-				(size 1 1)
-				(thickness 0.15)
-			)
-			(justify mirror)
-		)
-	)
 	(segment
 		(start 89.14 76.89)
@@
 	)
 	(segment
+		(start 102.96 108.77)
+		(end 75.59 108.77)
+		(width 0.5)
+		(layer "F.Cu")
+		(net 3)
+	)
+	(segment
+		(start 75.59 108.77)
+		(end 73.96 107.14)
+		(width 0.5)
+		(layer "F.Cu")
+		(net 3)
+	)
+	(segment
 		(start 76.44 59.11)
 		(end 76.328636 59.11)
@@
 		(net 3)
 	)
+	(segment
+		(start 108.5 103.23)
+		(end 102.96 108.77)
+		(width 0.5)
+		(layer "F.Cu")
+		(net 3)
+	)
+	(segment
+		(start 98.731 73.069)
+		(end 97.48 74.32)
+		(width 0.5)
+		(layer "B.Cu")
+		(net 3)
+	)
+	(segment
+		(start 97.48 59.08)
+		(end 98.731 60.331)
+		(width 0.5)
+		(layer "B.Cu")
+		(net 3)
+	)
+	(segment
+		(start 98.731 60.331)
+		(end 98.731 73.069)
+		(width 0.5)
+		(layer "B.Cu")
+		(net 3)
+	)
