File: PCB/_autosave-PCB-MTD.kicad_sch (KiCad schematic)
At the start: 26 parts, among them J1 Barrel_Jack_Switch, J2 Screw_Terminal_01x02, J9 Micro_SD_Card, U1 ESP32-S3-UNO, U2 R-78E5.0-1.0

Commit message: Add files via upload
Parts:
- C1, C2: footprint C_1206_3216Metric_Pad1.33x1.80mm_HandSolder -> Capacitor_SMD:CP_Elec_6.3x5.4
Changed lines of the file:
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@@
 			)
 		)
-		(property "Footprint" "C_1206_3216Metric_Pad1.33x1.80mm_HandSolder"
+		(property "Footprint" "Capacitor_SMD:CP_Elec_6.3x5.4"
 			(at 210.5152 139.7 0)
 			(effects
@@
 			)
 		)
+		(property "Field5" ""
+			(at 209.55 135.89 0)
+			(effects
+				(font
+					(size 1.27 1.27)
+				)
+				(hide yes)
+			)
+		)
 		(pin "1"
 		)
@@
 			)
 		)
-		(property "Footprint" "C_1206_3216Metric_Pad1.33x1.80mm_HandSolder"
+		(property "Footprint" "Capacitor_SMD:CP_Elec_6.3x5.4"
 			(at 304.4952 106.68 0)
 			(effects
