File: PCB/PCB-MTD.kicad_pcb (KiCad board)
At the start: 2 copper layers, 78.2 x 57.6 mm, 25 parts, among them J1 Barrel_Jack_Switch, J9 Micro_SD_Card, U1 ESP32-S3-UNO, U2 R-78E5.0-1.0

Commit message: Add files via upload
Parts:
- added J2: Screw_Terminal_01x02, TerminalBlock_Phoenix:TerminalBlock_Phoenix_MKDS-1,5-2-5.08_1x02_P5.08mm_Horizontal, F.Cu at (123.2, 59.8)
- added kibuzzard-69E8AB48: G***, kibuzzard-69E8AB48, F.Cu at (71.9, 89.6)
- added kibuzzard-69E8AB7B: G***, kibuzzard-69E8AB7B, F.Cu at (71.6, 98.4)
- added kibuzzard-69E8AB94: G***, kibuzzard-69E8AB94, F.Cu at (95.7, 89.2)
- added kibuzzard-69E8ABA4: G***, kibuzzard-69E8ABA4, F.Cu at (95.6, 98.2)
- added kibuzzard-69E8ABD2: G***, kibuzzard-69E8ABD2, F.Cu at (102.5, 84.3)
- added kibuzzard-69E8ABED: G***, kibuzzard-69E8ABED, F.Cu at (104.8, 81.6)
- added kibuzzard-69E8ABFE: G***, kibuzzard-69E8ABFE, F.Cu at (107.4, 81.4)
- added kibuzzard-69E8AC2D: G***, kibuzzard-69E8AC2D, F.Cu at (109.9, 81.6)
- added kibuzzard-69E8AC3C: G***, kibuzzard-69E8AC3C, F.Cu at (112.5, 81.6)
- added kibuzzard-69E8AC9A: G***, kibuzzard-69E8AC9A, F.Cu at (74.0, 104.8)
- added kibuzzard-69E8ACB2: G***, kibuzzard-69E8ACB2, F.Cu at (77.4, 104.8)
- added kibuzzard-69E8ACC9: G***, kibuzzard-69E8ACC9, F.Cu at (79.6, 104.8)
- added kibuzzard-69E8AD3B: G***, kibuzzard-69E8AD3B, F.Cu at (70.1, 66.7)
- added kibuzzard-69E8AD3B: G***, kibuzzard-69E8AD3B, F.Cu at (91.4, 66.4)
- added kibuzzard-69E8AD47: G***, kibuzzard-69E8AD47, F.Cu at (91.3, 69.2)
- added kibuzzard-69E8AD47: G***, kibuzzard-69E8AD47, F.Cu at (70.0, 69.3)
- added kibuzzard-69E8AD54: G***, kibuzzard-69E8AD54, F.Cu at (91.3, 71.9)
- added kibuzzard-69E8AD54: G***, kibuzzard-69E8AD54, F.Cu at (70.1, 71.9)
- added kibuzzard-69E8ADAF: G***, kibuzzard-69E8ADAF, F.Cu at (91.3, 74.5)
- added kibuzzard-69E8ADAF: G***, kibuzzard-69E8ADAF, F.Cu at (70.3, 74.6)
- added kibuzzard-69E8ADD5: G***, kibuzzard-69E8ADD5, F.Cu at (73.6, 59.0)
- added kibuzzard-69E8ADD5: G***, kibuzzard-69E8ADD5, F.Cu at (94.6, 59.0)
- added kibuzzard-69E8AE0E: G***, kibuzzard-69E8AE0E, F.Cu at (107.3, 92.3)
- added kibuzzard-69E8AE4C: G***, kibuzzard-69E8AE4C, F.Cu at (111.4, 93.9)
- added kibuzzard-69E8AE60: G***, kibuzzard-69E8AE60, F.Cu at (115.2, 87.0)
- added kibuzzard-69E8AE7F: G***, kibuzzard-69E8AE7F, F.Cu at (132.9, 78.3)
- added kibuzzard-69E8AE92: G***, kibuzzard-69E8AE92, F.Cu at (133.0, 66.2)
- added kibuzzard-69E8AEC7: G***, kibuzzard-69E8AEC7, F.Cu at (102.8, 79.8)
- added kibuzzard-69E8AEDA: G***, kibuzzard-69E8AEDA, F.Cu at (99.4, 88.3)
- added kibuzzard-69E8AEDA: G***, kibuzzard-69E8AEDA, F.Cu at (77.5, 84.5)
- added kibuzzard-69E8AEFD: G***, kibuzzard-69E8AEFD, F.Cu at (78.4, 82.5)
- added kibuzzard-69E8AF1C: G***, kibuzzard-69E8AF1C, F.Cu at (103.9, 90.0)
- added kibuzzard-69E8B027: G***, kibuzzard-69E8B027, F.Cu at (136.8, 78.4)
- added kibuzzard-69E8B027: G***, kibuzzard-69E8B027, F.Cu at (136.7, 66.2)
- added kibuzzard-69E8C7AB: G***, kibuzzard-69E8C7AB, F.Cu at (80.7, 69.0)
- added kibuzzard-69E8C7B2: G***, kibuzzard-69E8C7B2, F.Cu at (80.7, 71.8)
- added kibuzzard-69E8C7BE: G***, kibuzzard-69E8C7BE, F.Cu at (80.7, 74.5)
- added kibuzzard-69E8C827: G***, kibuzzard-69E8C827, F.Cu at (102.1, 74.4)
- added kibuzzard-69E8C830: G***, kibuzzard-69E8C830, F.Cu at (102.0, 72.0)
- added kibuzzard-69E8C83B: G***, kibuzzard-69E8C83B, F.Cu at (102.0, 69.2)
- added kibuzzard-69E8C8E3: G***, kibuzzard-69E8C8E3, F.Cu at (83.9, 107.0)
- C1, C2: footprint Capacitor_SMD:C_1206_3216Metric_Pad1.33x1.80mm_HandSolder -> Capacitor_SMD:CP_Elec_6.3x5.4
- moved C2 7.19 mm to (97.5, 83.2), turned to -90 degrees
- moved F1 6.26 mm to (129.0, 72.2), turned to 180 degrees
- moved C1 4.41 mm to (72.4, 81.9), turned to -90 degrees
- moved bas1 3.56 mm to (85.0, 95.8)
- moved haut1 3.56 mm to (85.0, 86.9)
- moved selectionner1 3.56 mm to (74.5, 95.8)
- moved retour1 3.56 mm to (74.5, 86.9)
- moved C5 0.66 mm to (102.8, 88.2)
Connections:
- F1 pad 2: Net-(F1-Pad2) -> Net-(J2-Pin_2)
- J1 pad 1: Net-(F1-Pad2) -> Net-(J2-Pin_1)
Routing:
- net GND: track 0.13 -> 92.8 mm
- net Net-(J2-Pin_1): track 0.00 -> 14.4 mm
- net Net-(F1-Pad2): track 14.1 -> 0.00 mm
- net Net-(J2-Pin_2): track 0.00 -> 12.8 mm
- net +5V: track 173.7 -> 178.1 mm
- net BTN_1: track 13.8 -> 10.6 mm
- net D2_DIR: track 77.5 -> 80.6 mm
- net BTN_2: track 34.0 -> 31.0 mm
- net BTN_4: track 13.7 -> 10.6 mm
- net BTN_3: track 23.2 -> 20.2 mm
- net 12VF: track 82.8 -> 84.5 mm
- net +3.3V: track 136.2 -> 136.7 mm
Other:
- board text removed: "${REFERENCE}"

Commit message: Add files via upload
Parts:
- moved R3 1.23 mm to (110.2, 90.1)
Connections:
- LCD1 pad 3: Net-(LCD1-Pin_3) -> SCL
- LCD1 pad 4: Net-(LCD1-Pin_4) -> SDA
- R2 pad 1: Net-(LCD1-Pin_4) -> +3.3V
- R3 pad 1: Net-(LCD1-Pin_3) -> +3.3V
- jumperD1 pad 1: +5V -> +3.3V
- jumperD1 pad 3: +5V -> +3.3V
- jumperD1 pad 5: +5V -> +3.3V
- jumperD2 pad 1: +5V -> +3.3V
- jumperD2 pad 3: +5V -> +3.3V
- jumperD2 pad 5: +5V -> +3.3V
Routing:
- net +3.3V: track 136.7 -> 176.7 mm
- net SCL: track 14.0 -> 30.4 mm
- net SDA: track 25.2 -> 37.0 mm
- net Net-(LCD1-Pin_3): track 5.75 -> 0.00 mm
- net Net-(LCD1-Pin_4): track 2.87 -> 0.00 mm
- net 12VF: track 84.5 -> 86.2 mm
- net +5V: track 178.1 -> 179.1 mm
- net D2_STEP: track 34.7 -> 34.2 mm

Commit message: Add files via upload
Parts:
- moved J9 1.20 mm to (134.2, 92.7)
Routing:
- net +3.3V: track 176.7 -> 182.7 mm
- net DAT0: track 27.2 -> 28.4 mm
- net CMD: track 22.5 -> 23.8 mm
- net CLK: track 20.1 -> 21.3 mm
- net DAT3/CD: track 69.1 -> 70.4 mm

Commit message: fix wiring problems
Connections:
- U1 pad 8: +5V -> 12VF
Routing:
- net +5V: track 179.1 -> 108.7 mm
- net 12VF: track 86.2 -> 137.3 mm
